Commit message: bobo1

File: rom_robot_class/bobo_description/urdf/bobo.urdf (robot description, URDF)
Before this commit: robot bobo_standalone, 13 links, 12 joints
Links:
- link base_link: geometry collision mesh filename=/ros2_ws/src/rom_robot_class/bobo_description/meshes/base_l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; visual mesh filename=/ros2_ws/src/rom_robot_class/bobo_description/meshes/base_l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
- link caster_back_left_link: geometry collision mesh filename=/ros2_ws/src/rom_robot_class/bobo_description/meshes/caster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; visual mesh filename=/ros2_ws/src/rom_robot_class/bobo_description/meshes/caster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
- link caster_back_right_link: geometry collision mesh filename=/ros2_ws/src/rom_robot_class/bobo_description/meshes/caster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; visual mesh filename=/ros2_ws/src/rom_robot_class/bobo_description/meshes/caster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
- link caster_front_left_link: geometry collision mesh filename=/ros2_ws/src/rom_robot_class/bobo_description/meshes/caster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; visual mesh filename=/ros2_ws/src/rom_robot_class/bobo_description/meshes/caster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
- link caster_front_right_link: geometry collision mesh filename=/ros2_ws/src/rom_robot_class/bobo_description/meshes/caster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; visual mesh filename=/ros2_ws/src/rom_robot_class/bobo_description/meshes/caster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
- link left_wheel_link: geometry collision mesh filename=/ros2_ws/src/rom_robot_class/bobo_description/meshes/wheel_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; visual mesh filename=/ros2_ws/src/rom_robot_class/bobo_description/meshes/wheel_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
- link right_wheel_link: geometry collision mesh filename=/ros2_ws/src/rom_robot_class/bobo_description/meshes/wheel_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; visual mesh filename=/ros2_ws/src/rom_robot_class/bobo_description/meshes/wheel_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
Joints:
- removed joint wheel_left_joint
- removed joint wheel_right_joint
- added joint left_wheel_joint: type continuous, parent base_link, child left_wheel_link, origin xyz=-0.0005 0.17971 0.0854 rpy=0 0 0, axis 0 -1 0
- added joint right_wheel_joint: type continuous, parent base_link, child right_wheel_link, origin xyz=-0.0005 -0.17971 0.0854 rpy=0 0 0, axis 0 -1 0
- joint caster_back_left_joint: type continuous -> fixed
- joint caster_back_right_joint: type continuous -> fixed
- joint caster_front_left_joint: type continuous -> fixed
- joint caster_front_right_joint: type continuous -> fixed

File: rom_robot_class/bobo_description/urdf/sim_lidar.xacro (robot description, xacro)
@@ -27,5 +27,5 @@
                 </ros>
                 <output_type>sensor_msgs/LaserScan</output_type>
-                <frame_name>lidar</frame_name>
+                <frame_name>laser_link</frame_name>
             </plugin>
         </sensor>

File: rom_robot_class/bobo_description/urdf/sim_robot2.xacro (robot description, xacro)
@@ -51,5 +51,5 @@
   </link>
   <link
-    name="wheel_right_link">
+    name="right_wheel_link">
     <inertial>
       <origin
@@ -91,5 +91,5 @@
   </link>
   <joint
-    name="wheel_right_joint"
+    name="right_wheel_joint"
     type="continuous">
     <origin
@@ -99,10 +99,10 @@
       link="base_link" />
     <child
-      link="wheel_right_link" />
+      link="right_wheel_link" />
     <axis
       xyz="0 -1 0" />
   </joint>
   <link
-    name="wheel_left_link">
+    name="left_wheel_link">
     <inertial>
       <origin
@@ -144,5 +144,5 @@
   </link>
   <joint
-    name="wheel_left_joint"
+    name="left_wheel_joint"
     type="continuous">
     <origin
@@ -152,5 +152,5 @@
       link="base_link" />
     <child
-      link="wheel_left_link" />
+      link="left_wheel_link" />
     <axis
       xyz="0 -1 0" />
@@ -198,5 +198,5 @@
   <joint
     name="caster_front_right_joint"
-    type="continuous">
+    type="fixed">
     <origin
       xyz="0.16676 -0.077762 0.016"
@@ -251,5 +251,5 @@
   <joint
     name="caster_front_left_joint"
-    type="continuous">
+    type="fixed">
     <origin
       xyz="0.16676 0.077762 0.016"
@@ -304,5 +304,5 @@
   <joint
     name="caster_back_left_joint"
-    type="continuous">
+    type="fixed">
     <origin
       xyz="-0.16676 0.077762 0.016"
@@ -357,5 +357,5 @@
   <joint
     name="caster_back_right_joint"
-    type="continuous">
+    type="fixed">
     <origin
       xyz="-0.16676 -0.077762 0.016"
@@ -381,5 +381,5 @@
           <box size="0.05 0.05 0.05"/>
         </geometry>
-        <material name="grey_blue"/>
+        <material name="red"/>
       </visual>
       <collision>
@@ -409,5 +409,5 @@
           <box size="0.03 0.02 0.02"/>
         </geometry>
-        <material name="red"/>
+        <material name="green"/>
       </visual>
   </link>
@@ -424,5 +424,5 @@
           <box size="0.03 0.02 0.02"/>
         </geometry>
-        <material name="orange"/>
+        <material name="blue"/>
       </visual>
   </link>
@@ -439,5 +439,5 @@
           <box size="0.03 0.02 0.02"/>
         </geometry>
-        <material name="orange"/>
+        <material name="blue"/>
       </visual>
   </link>
@@ -454,5 +454,5 @@
           <box size="0.03 0.02 0.02"/>
         </geometry>
-        <material name="orange"/>
+        <material name="blue"/>
       </visual>
   </link>

File: rom_robot_class/bobo_description/urdf/sim_robot2_complete.urdf.xacro (robot description, xacro)
@@ -3,6 +3,6 @@
     <xacro:arg name="prefix" default="" />
     <xacro:include filename="$(find bobo_description)/urdf/$(env BOBO_MODEL).xacro" />
-    <!-- <xacro:include filename="$(env BOBO_MODEL)_ros2_control.xacro" />
-    <xacro:include filename="sim_lidar.xacro" /> -->
+    <xacro:include filename="$(env BOBO_MODEL)_ros2_control.xacro" />
+    <xacro:include filename="sim_lidar.xacro" />
     <!--xacro:include filename="sim_camera.xacro" /-->
     <!-- <xacro:include filename="sim_camera3d.xacro" /> -->

File: rom_robot_class/bobo_description/urdf/sim_robot2_ros2_control.xacro (robot description, xacro)
@@ -5,5 +5,5 @@
             <plugin>gazebo_ros2_control/GazeboSystem</plugin>
         </hardware>
-        <joint name="wheel_left_joint">
+        <joint name="left_wheel_joint">
             <command_interface name="velocity">
                 <param name="min">-500</param>
@@ -13,5 +13,5 @@
             <state_interface name="position"/>
         </joint>
-        <joint name="wheel_right_joint">
+        <joint name="right_wheel_joint">
             <command_interface name="velocity">
                 <param name="min">-500</param>
@@ -26,5 +26,5 @@
             <robot_param>robot_description</robot_param>
             <robot_param_node>robot_state_publisher</robot_param_node>
-            <parameters>$(find bobo_description)/config/my_controllers.yaml</parameters>
+            <parameters>$(find bobo_description)/sim_config/my_controllers.yaml</parameters>
             <!-- Output -->
             <odometry_frame>odom</odometry_frame>

Commit message: update

File: rom_robot_class/bobo_description/urdf/bobo.urdf (robot description, URDF)
Before this commit: robot bobo_standalone, 13 links, 12 joints
Links:
- added link camera_link_optical
- added link camera_link_optical_left
- added link camera_link_optical_right
Joints:
- added joint camera_optical_joint: type fixed, parent cam3d_top_link, child camera_link_optical, origin xyz=0 0 0 rpy=-1.57075 0 -1.57075
- added joint camera_optical_joint_left: type fixed, parent cam3d_left_link, child camera_link_optical_left, origin xyz=0 0 0 rpy=-1.57075 0 -1.57075
- added joint camera_optical_joint_right: type fixed, parent cam3d_right_link, child camera_link_optical_right, origin xyz=0 0 0 rpy=-1.57075 0 -1.57075

File: rom_robot_class/bobo_description/urdf/sim_camera3d _left.xacro (robot description, xacro)
@@ -1,14 +1,14 @@
 <?xml version="1.0"?>
 <robot xmlns:xacro="http://www.ros.org/wiki/xacro">
-  <!-- TOP CAMERA -->
-  <joint name="camera_optical_joint" type="fixed">
-        <parent link="cam3d_top_link"/>
-        <child link="camera_link_optical"/>
+</robot> <!-- LEFT CAMERA -->
+  <joint name="camera_optical_joint_left" type="fixed">
+        <parent link="cam3d_left_link"/>
+        <child link="camera_link_optical_left"/>
         <origin xyz="0 0 0" rpy="-1.57075 0 -1.57075"/> <!-- ${-pi/2} -->
     </joint>
-    <link name="camera_link_optical"></link>
-    <gazebo reference="cam3d_top_link">
+    <link name="camera_link_optical_left"></link>
+    <gazebo reference="cam3d_left_link">
         <material>Gazebo/Blue</material>
-        <sensor name="camera_top" type="depth">
+        <sensor name="camera_left" type="depth">
             <pose>0 0 0 0 0 0</pose>
             <visualize>true</visualize>
@@ -26,6 +26,6 @@
                 </clip>
             </camera>
-            <plugin name="camera_controller_top" filename="libgazebo_ros_camera.so">
-                <frame_name>camera_link_optical</frame_name>
+            <plugin name="camera_controller_left" filename="libgazebo_ros_camera.so">
+                <frame_name>camera_link_optical_left</frame_name>
                 <min_depth>0.1</min_depth>
                 <max_depth>50</max_depth>

File: rom_robot_class/bobo_description/urdf/sim_camera3d _right.xacro (robot description, xacro)
@@ -1,14 +1,14 @@
 <?xml version="1.0"?>
 <robot xmlns:xacro="http://www.ros.org/wiki/xacro">
-  <!-- TOP CAMERA -->
-  <joint name="camera_optical_joint" type="fixed">
-        <parent link="cam3d_top_link"/>
-        <child link="camera_link_optical"/>
+      <!-- RIGHT CAMERA -->
+  <joint name="camera_optical_joint_right" type="fixed">
+        <parent link="cam3d_right_link"/>
+        <child link="camera_link_optical_right"/>
         <origin xyz="0 0 0" rpy="-1.57075 0 -1.57075"/> <!-- ${-pi/2} -->
     </joint>
-    <link name="camera_link_optical"></link>
-    <gazebo reference="cam3d_top_link">
+    <link name="camera_link_optical_right"></link>
+    <gazebo reference="cam3d_right_link_right">
         <material>Gazebo/Blue</material>
-        <sensor name="camera_top" type="depth">
+        <sensor name="camera_right" type="depth">
             <pose>0 0 0 0 0 0</pose>
             <visualize>true</visualize>
@@ -26,6 +26,6 @@
                 </clip>
             </camera>
-            <plugin name="camera_controller_top" filename="libgazebo_ros_camera.so">
-                <frame_name>camera_link_optical</frame_name>
+            <plugin name="camera_controller_right" filename="libgazebo_ros_camera.so">
+                <frame_name>camera_link_optical_right</frame_name>
                 <min_depth>0.1</min_depth>
                 <max_depth>50</max_depth>

File: rom_robot_class/bobo_description/urdf/sim_robot2_complete.urdf.xacro (robot description, xacro)
@@ -6,4 +6,6 @@
     <xacro:include filename="sim_lidar.xacro" />
     <!--xacro:include filename="sim_camera.xacro" /-->
-    <!-- <xacro:include filename="sim_camera3d.xacro" /> -->
+    <xacro:include filename="sim_camera3d.xacro" />
+    <!-- <xacro:include filename="sim_camera3d_left.xacro" />
+    <xacro:include filename="sim_camera3d_right.xacro" /> -->
 </robot>
