Commit message: update

File: rom_robot_class/bobo_description/urdf/bobo.urdf (robot description, URDF)
Before this commit: robot bobo_standalone, 16 links, 15 joints
Links:
- removed link camera_link_optical_left
- removed link camera_link_optical_right
- removed link caster_back_left_link
- removed link caster_back_right_link
- removed link caster_front_left_link
- removed link caster_front_right_link
- added link back_left_caster_link, mass 0.051978; collision mesh filename=/ros2_ws/src/rom_robot_class/bobo_description/meshes/back_l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; visual mesh filename=/ros2_ws/src/rom_robot_class/bobo_description/meshes/back_l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
- added link back_left_caster_wheel_link, mass 4.2523; collision mesh filename=/ros2_ws/src/rom_robot_class/bobo_description/meshes/back_l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; visual mesh filename=/ros2_ws/src/rom_robot_class/bobo_description/meshes/back_l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
- added link back_right_caster_link, mass 0.051978; collision mesh filename=/ros2_ws/src/rom_robot_class/bobo_description/meshes/back_r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; visual mesh filename=/ros2_ws/src/rom_robot_class/bobo_description/meshes/back_r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
- added link back_right_caster_wheel_link, mass 0.010387; collision mesh filename=/ros2_ws/src/rom_robot_class/bobo_description/meshes/back_r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; visual mesh filename=/ros2_ws/src/rom_robot_class/bobo_description/meshes/back_r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
- added link front_left_caster_link, mass 0.051978; collision mesh filename=/ros2_ws/src/rom_robot_class/bobo_description/meshes/front_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; visual mesh filename=/ros2_ws/src/rom_robot_class/bobo_description/meshes/front_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
- added link front_left_caster_wheel_link, mass 0.010387; collision mesh filename=/ros2_ws/src/rom_robot_class/bobo_description/meshes/front_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; visual mesh filename=/ros2_ws/src/rom_robot_class/bobo_description/meshes/front_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
- added link front_right_caster_link, mass 0.051978; collision mesh filename=/ros2_ws/src/rom_robot_class/bobo_description/meshes/front_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; visual mesh filename=/ros2_ws/src/rom_robot_class/bobo_description/meshes/front_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
- added link front_right_caster_wheel_link, mass 0.010387; collision mesh filename=/ros2_ws/src/rom_robot_class/bobo_description/meshes/front_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; visual mesh filename=/ros2_ws/src/rom_robot_class/bobo_description/meshes/front_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
- link base_link: mass 1.9421 -> 1.7335
- link left_wheel_link: mass 1.13468316605061 -> 1.1347; geometry collision mesh filename=/ros2_ws/src/rom_robot_class/bobo_description/meshes/left_w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; visual mesh filename=/ros2_ws/src/rom_robot_class/bobo_description/meshes/left_w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
- link right_wheel_link: mass 1.13468316605061 -> 1.1347; geometry collision mesh filename=/ros2_ws/src/rom_robot_class/bobo_description/meshes/right_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; visual mesh filename=/ros2_ws/src/rom_robot_class/bobo_description/meshes/right_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
Joints:
- removed joint camera_optical_joint_left
- removed joint camera_optical_joint_right
- removed joint caster_back_left_joint
- removed joint caster_back_right_joint
- removed joint caster_front_left_joint
- removed joint caster_front_right_joint
- added joint back_left_caster_joint: type fixed, parent base_link, child back_left_caster_link, origin xyz=-0.16676 0.077762 0.1 rpy=0 0 0, axis 0 0 1, limit lower=0 upper=0 effort=0 velocity=0
- added joint back_left_caster_wheel_joint: type fixed, parent back_left_caster_link, child back_left_caster_wheel_link, origin xyz=0 0 -0.084 rpy=0 0 0.436332312998583, axis -0.392612736878362 -0.919703886498737 0
- added joint back_right_caster_joint: type fixed, parent base_link, child back_right_caster_link, origin xyz=-0.16676 -0.077762 0.1 rpy=0 0 0, axis 0 0 1, limit lower=0 upper=0 effort=0 velocity=0
- added joint back_right_caster_wheel_joint: type fixed, parent back_right_caster_link, child back_right_caster_wheel_link, origin xyz=0 0 -0.0839999999999996 rpy=0 0 -0.436332312998583, axis 0.430004766049687 -0.902826617449084 0
- added joint front_left_caster_joint: type fixed, parent base_link, child front_left_caster_link, origin xyz=0.16676 0.077762 0.1 rpy=0 0 0, axis 0 0 -1, limit lower=0 upper=0 effort=0 velocity=0
- added joint front_left_caster_wheel_joint: type fixed, parent front_left_caster_link, child front_left_caster_wheel_link, origin xyz=0 0 -0.0840000000000001 rpy=0 0 -0.436332312998583, axis -0.450731309052789 0.892659670333302 0
- added joint front_right_caster_joint: type fixed, parent base_link, child front_right_caster_link, origin xyz=0.16676 -0.077762 0.1 rpy=0 0 0, axis 0 0 -1, limit lower=0 upper=0 effort=0 velocity=0
- added joint front_right_caster_wheel_joint: type fixed, parent front_right_caster_link, child front_right_caster_wheel_link, origin xyz=0 0 -0.084 rpy=0 0 0.436332312998583, axis 0.420626471111868 0.907233912395242 0
- joint left_wheel_joint: axis 0 -1 0 -> 0 1 0; origin xyz=-0.0005 0.17971 0.0854 rpy=0 0 0 -> xyz=-0.000500000000000396 0.179709309933579 0.085 rpy=0 0 0
- joint right_wheel_joint: axis 0 -1 0 -> 0 1 0; origin xyz=-0.0005 -0.17971 0.0854 rpy=0 0 0 -> xyz=-0.000499999999999182 -0.179709309933579 0.085 rpy=0 0 0

File: rom_robot_class/bobo_description/urdf/sim_lidar.xacro (robot description, xacro)
@@ -17,5 +17,5 @@
                 </scan>
                 <range>
-                    <min>0.05</min><!-- 0.3 -->
+                    <min>0.5</min><!-- 0.3 -->
                     <max>12</max><!-- 12 -->
                     <resolution>0.01</resolution>

File: rom_robot_class/bobo_description/urdf/sim_robot2.xacro (robot description, xacro)
@@ -7,22 +7,23 @@
   <link name="base_footprint"/>
     <joint name="base_joint" type="fixed">
-      <origin xyz="0 0 0" rpy="0 0 0" />
-      <parent link="base_footprint"/>
-      <child link="base_link" />
+    <origin xyz="0 0 0" rpy="0 0 0" />
+    <parent link="base_footprint"/>
+    <child link="base_link" />
     </joint>
-  <link name="base_link">
-    <inertial>
-      <origin
-        xyz="0.0046524 -1.2029E-05 0.18162"
-        rpy="0 0 0" />
-      <mass
-        value="1.9421" />
-      <inertia
-        ixx="0.016249"
-        ixy="-2.6352E-08"
+    <link
+    name="base_link">
+    <inertial>
+      <origin
+        xyz="0.0052125 -1.3478E-05 0.19649"
+        rpy="0 0 0" />
+      <mass
+        value="1.7335" />
+      <inertia
+        ixx="0.016138"
+        ixy="-2.6556E-08"
         ixz="-0.00032505"
-        iyy="0.019076"
+        iyy="0.018981"
         iyz="2.2146E-08"
-        izz="0.031848" />
+        izz="0.031833" />
     </inertial>
     <visual>
@@ -54,23 +55,23 @@
     <inertial>
       <origin
-        xyz="-6.88469101173261E-10 0.00261076778922063 1.46539359813236E-09"
-        rpy="0 0 0" />
-      <mass
-        value="1.13468316605061" />
-      <inertia
-        ixx="0.00214377737472316"
-        ixy="1.35474255028293E-09"
-        ixz="-1.11198689477431E-11"
-        iyy="0.00371288553259231"
-        iyz="-1.63769629423567E-09"
-        izz="0.00214377737749942" />
-    </inertial>
-    <visual>
-      <origin
-        xyz="0 0 0"
-        rpy="0 0 0" />
-      <geometry>
-        <mesh
-          filename="package://bobo_description/meshes/wheel_right_link.STL" />
+        xyz="-1.6048E-09 0.0026108 -2.1412E-10"
+        rpy="0 0 0" />
+      <mass
+        value="1.1347" />
+      <inertia
+        ixx="0.0021438"
+        ixy="1.9702E-09"
+        ixz="8.2955E-12"
+        iyy="0.0037129"
+        iyz="7.9733E-10"
+        izz="0.0021438" />
+    </inertial>
+    <visual>
+      <origin
+        xyz="0 0 0"
+        rpy="0 0 0" />
+      <geometry>
+        <mesh
+          filename="package://bobo_description/meshes/right_wheel_link.STL" />
       </geometry>
       <material
@@ -86,5 +87,5 @@
       <geometry>
         <mesh
-          filename="package://bobo_description/meshes/wheel_right_link.STL" />
+          filename="package://bobo_description/meshes/right_wheel_link.STL" />
       </geometry>
     </collision>
@@ -94,5 +95,5 @@
     type="continuous">
     <origin
-      xyz="-0.0005 -0.17971 0.0854"
+      xyz="-0.000499999999999182 -0.179709309933579 0.085"
       rpy="0 0 0" />
     <parent
@@ -101,5 +102,5 @@
       link="right_wheel_link" />
     <axis
-      xyz="0 -1 0" />
+      xyz="0 1 0" />
   </joint>
   <link
@@ -107,23 +108,23 @@
     <inertial>
       <origin
-        xyz="1.61277113885916E-09 -0.00261076778922059 1.42610201425697E-10"
-        rpy="0 0 0" />
-      <mass
-        value="1.13468316605061" />
-      <inertia
-        ixx="0.00214377738646834"
-        ixy="2.09699277269092E-09"
-        ixz="-4.27898719562988E-12"
-        iyy="0.00371288553259229"
-        iyz="-3.46407025976004E-10"
-        izz="0.00214377736575422" />
-    </inertial>
-    <visual>
-      <origin
-        xyz="0 0 0"
-        rpy="0 0 0" />
-      <geometry>
-        <mesh
-          filename="package://bobo_description/meshes/wheel_left_link.STL" />
+        xyz="1.4724E-09 -0.0026108 -6.7344E-10"
+        rpy="0 0 0" />
+      <mass
+        value="1.1347" />
+      <inertia
+        ixx="0.0021438"
+        ixy="1.6515E-09"
+        ixz="-1.1089E-11"
+        iyy="0.0037129"
+        iyz="-1.3379E-09"
+        izz="0.0021438" />
+    </inertial>
+    <visual>
+      <origin
+        xyz="0 0 0"
+        rpy="0 0 0" />
+      <geometry>
+        <mesh
+          filename="package://bobo_description/meshes/left_wheel_link.STL" />
       </geometry>
       <material
@@ -139,5 +140,5 @@
       <geometry>
         <mesh
-          filename="package://bobo_description/meshes/wheel_left_link.STL" />
+          filename="package://bobo_description/meshes/left_wheel_link.STL" />
       </geometry>
     </collision>
@@ -147,5 +148,5 @@
     type="continuous">
     <origin
-      xyz="-0.0005 0.17971 0.0854"
+      xyz="-0.000500000000000396 0.179709309933579 0.085"
       rpy="0 0 0" />
     <parent
@@ -154,29 +155,87 @@
       link="left_wheel_link" />
     <axis
-      xyz="0 -1 0" />
-  </joint>
-  <link
-    name="caster_front_right_link">
-    <inertial>
-      <origin
-        xyz="-1.38777878078145E-17 -1.38777878078145E-17 -2.77555756156289E-17"
-        rpy="0 0 0" />
-      <mass
-        value="0.0103871549572359" />
-      <inertia
-        ixx="9.76068238842766E-07"
-        ixy="4.37487850150777E-08"
-        ixz="4.36668756326797E-23"
-        iyy="1.47229853084168E-06"
-        iyz="5.40669622917979E-22"
-        izz="9.72240768629191E-07" />
-    </inertial>
-    <visual>
-      <origin
-        xyz="0 0 0"
-        rpy="0 0 0" />
-      <geometry>
-        <mesh
-          filename="package://bobo_description/meshes/caster_front_right_link.STL" />
+      xyz="0 1 0" />
+  </joint>
+  <link
+    name="front_right_caster_link">
+    <inertial>
+      <origin
+        xyz="-1.3878E-16 1.3791E-16 -0.045367"
+        rpy="0 0 0" />
+      <mass
+        value="0.051978" />
+      <inertia
+        ixx="2.8149E-05"
+        ixy="2.1927E-09"
+        ixz="-6.8047E-20"
+        iyy="2.7151E-05"
+        iyz="-1.1119E-21"
+        izz="8.6419E-06" />
+    </inertial>
+    <visual>
+      <origin
+        xyz="0 0 0"
+        rpy="0 0 0" />
+      <geometry>
+        <mesh
+          filename="package://bobo_description/meshes/front_right_caster_link.STL" />
+      </geometry>
+      <material
+        name="">
+        <color
+          rgba="0.79216 0.81961 0.93333 1" />
+      </material>
+    </visual>
+    <collision>
+      <origin
+        xyz="0 0 0"
+        rpy="0 0 0" />
+      <geometry>
+        <mesh
+          filename="package://bobo_description/meshes/front_right_caster_link.STL" />
+      </geometry>
+    </collision>
+  </link>
+  <joint
+    name="front_right_caster_joint"
+    type="fixed">
+    <origin
+      xyz="0.16676 -0.077762 0.1"
+      rpy="0 0 0" />
+    <parent
+      link="base_link" />
+    <child
+      link="front_right_caster_link" />
+    <axis
+      xyz="0 0 -1" />
+    <limit
+      lower="0"
+      upper="0"
+      effort="0"
+      velocity="0" />
+  </joint>
+  <link
+    name="front_right_caster_wheel_link">
+    <inertial>
+      <origin
+        xyz="0 -6.9389E-18 2.7756E-17"
+        rpy="0 0 0" />
+      <mass
+        value="0.010387" />
+      <inertia
+        ixx="1.0614E-06"
+        ixy="1.9229E-07"
+        ixz="1.2963E-13"
+        iyy="1.387E-06"
+        iyz="2.7958E-13"
+        izz="9.7224E-07" />
+    </inertial>
+    <visual>
+      <origin
+        xyz="0 0 0"
+        rpy="0 0 0" />
+      <geometry>
+        <mesh
+          filename="package://bobo_description/meshes/front_right_caster_wheel_link.STL" />
       </geometry>
       <material
@@ -192,44 +251,102 @@
       <geometry>
         <mesh
-          filename="package://bobo_description/meshes/caster_front_right_link.STL" />
-      </geometry>
-    </collision>
-  </link>
-  <joint
-    name="caster_front_right_joint"
+          filename="package://bobo_description/meshes/front_right_caster_wheel_link.STL" />
+      </geometry>
+    </collision>
+  </link>
+  <joint
+    name="front_right_caster_wheel_joint"
     type="fixed">
     <origin
-      xyz="0.16676 -0.077762 0.016"
-      rpy="0 0 0.43633" />
+      xyz="0 0 -0.084"
+      rpy="0 0 0.436332312998583" />
+    <parent
+      link="front_right_caster_link" />
+    <child
+      link="front_right_caster_wheel_link" />
+    <axis
+      xyz="0.420626471111868 0.907233912395242 0" />
+  </joint>
+  <link
+    name="front_left_caster_link">
+    <inertial>
+      <origin
+        xyz="-5.5511E-17 -2.7756E-17 -0.045367"
+        rpy="0 0 0" />
+      <mass
+        value="0.051978" />
+      <inertia
+        ixx="2.8148E-05"
+        ixy="3.1177E-08"
+        ixz="-6.9468E-20"
+        iyy="2.7152E-05"
+        iyz="-1.5896E-21"
+        izz="8.6419E-06" />
+    </inertial>
+    <visual>
+      <origin
+        xyz="0 0 0"
+        rpy="0 0 0" />
+      <geometry>
+        <mesh
+          filename="package://bobo_description/meshes/front_left_caster_link.STL" />
+      </geometry>
+      <material
+        name="">
+        <color
+          rgba="0.79216 0.81961 0.93333 1" />
+      </material>
+    </visual>
+    <collision>
+      <origin
+        xyz="0 0 0"
+        rpy="0 0 0" />
+      <geometry>
+        <mesh
+          filename="package://bobo_description/meshes/front_left_caster_link.STL" />
+      </geometry>
+    </collision>
+  </link>
+  <joint
+    name="front_left_caster_joint"
+    type="fixed">
+    <origin
+      xyz="0.16676 0.077762 0.1"
+      rpy="0 0 0" />
     <parent
       link="base_link" />
     <child
-      link="caster_front_right_link" />
-    <axis
-      xyz="-0.087156 -0.99619 0" />
-  </joint>
-  <link
-    name="caster_front_left_link">
-    <inertial>
-      <origin
-        xyz="-1.38777878078145E-17 -5.55111512312578E-17 0"
-        rpy="0 0 0" />
-      <mass
-        value="0.0103871549572359" />
-      <inertia
-        ixx="9.76068447320134E-07"
-        ixy="-4.37499673489831E-08"
-        ixz="3.49242855259726E-23"
-        iyy="1.47229832236431E-06"
-        iyz="-6.51906793689185E-22"
-        izz="9.72240768629191E-07" />
-    </inertial>
-    <visual>
-      <origin
-        xyz="0 0 0"
-        rpy="0 0 0" />
-      <geometry>
-        <mesh
-          filename="package://bobo_description/meshes/caster_front_left_link.STL" />
+      link="front_left_caster_link" />
+    <axis
+      xyz="0 0 -1" />
+    <limit
+      lower="0"
+      upper="0"
+      effort="0"
+      velocity="0" />
+  </joint>
+  <link
+    name="front_left_caster_wheel_link">
+    <inertial>
+      <origin
+        xyz="0 0 0"
+        rpy="0 0 0" />
+      <mass
+        value="0.010387" />
+      <inertia
+        ixx="1.0746E-06"
+        ixy="-2.0274E-07"
+        ixz="1.5821E-13"
+        iyy="1.3738E-06"
+        iyz="-3.1332E-13"
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