Commit message: gazebo worlds ok in container

File: simulation_packages/bobo_description/urdf/bobo.urdf (robot description, URDF)
Before this commit: robot bobo_standalone, 18 links, 17 joints
Links:
- link back_left_caster_link: geometry collision mesh filename=/bobo_ws/src/simulation_packages/bobo_description/meshes/ba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; visual mesh filename=/bobo_ws/src/simulation_packages/bobo_description/meshes/ba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
- link back_left_caster_wheel_link: geometry collision mesh filename=/bobo_ws/src/simulation_packages/bobo_description/meshes/ba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; visual mesh filename=/bobo_ws/src/simulation_packages/bobo_description/meshes/ba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
- link back_right_caster_link: geometry collision mesh filename=/bobo_ws/src/simulation_packages/bobo_description/meshes/ba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; visual mesh filename=/bobo_ws/src/simulation_packages/bobo_description/meshes/ba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
- link back_right_caster_wheel_link: geometry collision mesh filename=/bobo_ws/src/simulation_packages/bobo_description/meshes/ba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; visual mesh filename=/bobo_ws/src/simulation_packages/bobo_description/meshes/ba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
- link base_link: geometry collision mesh filename=/bobo_ws/src/simulation_packages/bobo_description/meshes/ba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; visual mesh filename=/bobo_ws/src/simulation_packages/bobo_description/meshes/ba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
- link front_left_caster_link: geometry collision mesh filename=/bobo_ws/src/simulation_packages/bobo_description/meshes/fr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; visual mesh filename=/bobo_ws/src/simulation_packages/bobo_description/meshes/fr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
- link front_left_caster_wheel_link: geometry collision mesh filename=/bobo_ws/src/simulation_packages/bobo_description/meshes/fr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; visual mesh filename=/bobo_ws/src/simulation_packages/bobo_description/meshes/fr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
- link front_right_caster_link: geometry collision mesh filename=/bobo_ws/src/simulation_packages/bobo_description/meshes/fr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; visual mesh filename=/bobo_ws/src/simulation_packages/bobo_description/meshes/fr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
- link front_right_caster_wheel_link: geometry collision mesh filename=/bobo_ws/src/simulation_packages/bobo_description/meshes/fr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; visual mesh filename=/bobo_ws/src/simulation_packages/bobo_description/meshes/fr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
- link left_wheel_link: geometry collision mesh filename=/bobo_ws/src/simulation_packages/bobo_description/meshes/le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; visual mesh filename=/bobo_ws/src/simulation_packages/bobo_description/meshes/le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
- link right_wheel_link: geometry collision mesh filename=/bobo_ws/src/simulation_packages/bobo_description/meshes/ri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; visual mesh filename=/bobo_ws/src/simulation_packages/bobo_description/meshes/ri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
