Commit message: update

File: simulation_packages/romrobots_description/urdf/bobo.xacro (robot description, xacro)
@@ -1,5 +1,5 @@
 <?xml version="1.0" ?>
 <robot name="robot" xmlns:xacro="http://ros.org/wiki/xacro">
-  <xacro:include filename="$(find romrobots_description)/urdf/bobo_common_properties.urdf.xacro"/>
+  <xacro:include filename="$(find romrobots_description)/urdf/common_properties.urdf.xacro"/>
   <xacro:macro name="robot">
     <link name="base_footprint"/>
@@ -93,58 +93,54 @@
       </inertial>
     </link>
-    <joint name="caster_front_joint" type="fixed">
-      <parent link="base_link"/>
-      <child link="caster_front_link"/>
-      <origin xyz="0.17 0.0 0.0195" rpy="${-M_PI/2} 0 0"/>
-    </joint>
-    <link name="caster_front_link">
-      <visual>
-        <geometry>
-          <cylinder length="0.0276" radius="0.035"/>
-        </geometry>
-        <origin xyz="0 0 0" rpy="0 0 0"/>
-        <material name="black"/>
-      </visual>
-      <collision>
-        <geometry>
-          <sphere radius="0.035"/>
-        </geometry>
-        <origin rpy="0 0 0" xyz="0 0 0"/>
-      </collision>
-      <inertial>
-        <mass value="0.01" />
-        <origin xyz="0 0 0" />
-        <inertia ixx="0.001" ixy="0.0" ixz="0.0"
-                 iyy="0.001" iyz="0.0"
-                 izz="0.001" />
-      </inertial>
-    </link>
-    <joint name="caster_back_joint" type="fixed">
-      <parent link="base_link"/>
-      <child link="caster_back_link"/>
-      <origin xyz="-0.17 0.0 0.015" rpy="${-M_PI/2} 0 0"/>
-    </joint>
-    <link name="caster_back_link">
-      <visual>
-        <geometry>
-          <cylinder length="0.0276" radius="0.035"/>
-        </geometry>
-        <origin xyz="0 0 0" rpy="0 0 0"/>
-        <material name="black"/>
-      </visual>
-      <collision>
-        <geometry>
-          <sphere radius="0.035"/>
-        </geometry>
-        <origin rpy="0 0 0" xyz="0 0 0"/>
-      </collision>
-      <inertial>
-        <mass value="0.01" />
-        <origin xyz="0 0 0" />
-        <inertia ixx="0.001" ixy="0.0" ixz="0.0"
-                 iyy="0.001" iyz="0.0"
-                 izz="0.001" />
-      </inertial>
-    </link>
+<!-- NEW CASTER -->
+  <link name="front_caster_ball">
+    <inertial>
+      <mass value="0.1"/>  <!-- Adjust the mass as per your robot's specs -->
+      <inertia ixx="0.001" iyy="0.001" izz="0.001" ixy="0.0" ixz="0.0" iyz="0.0"/>
+    </inertial>
+    <visual>
+      <geometry>
+        <sphere radius="0.02"/>  <!-- Radius of the caster ball -->
+      </geometry>
+      <material name="grey">
+        <color rgba="0.5 0.5 0.5 1.0"/>
+      </material>
+    </visual>
+    <collision>
+      <geometry>
+        <sphere radius="0.02"/>  <!-- Same radius as the visual element -->
+      </geometry>
+    </collision>
+  </link>
+  <joint name="front_caster_ball_joint" type="fixed">
+    <parent link="base_link"/>
+    <child link="front_caster_ball"/>
+    <origin xyz="0.16676 0 0.01" rpy="0 0 0"/>  <!-- z axis  -->
+  </joint>
+  <link name="back_caster_ball">
+    <inertial>
+      <mass value="0.1"/>  <!-- Adjust the mass as per your robot's specs -->
+       <inertia ixx="0.001" iyy="0.001" izz="0.001" ixy="0.0" ixz="0.0" iyz="0.0"/>
+    </inertial>
+    <visual>
+      <geometry>
+        <sphere radius="0.02"/>  <!-- Radius of the caster ball -->
+      </geometry>
+      <material name="grey">
+        <color rgba="0.5 0.5 0.5 1.0"/>
+      </material>
+    </visual>
+    <collision>
+      <geometry>
+        <sphere radius="0.02"/>  <!-- Same radius as the visual element -->
+      </geometry>
+    </collision>
+  </link>
+  <joint name="back_caster_ball_joint" type="fixed">
+    <parent link="base_link"/>
+    <child link="back_caster_ball"/>
+    <origin xyz="-0.16676 0 0.01" rpy="0 0 0"/>  <!-- z axis  -->
+  </joint>
+<!-- caster end -->
     <joint name="imu_joint" type="fixed">
       <parent link="base_link"/>

File: simulation_packages/romrobots_description/urdf/yoyo.urdf (robot description, URDF)
Before this commit: robot bobo_standalone, 10 links, 9 joints
Links:
- link base_link: mass 2.4 -> 1.7335; geometry collision mesh filename=/home/mr_robot/test_ws/src/bobo_simulation/simulation_packa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; visual mesh filename=/home/mr_robot/test_ws/src/bobo_simulation/simulation_packa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
- link left_wheel_link: mass 0.01 -> 1.1347; geometry collision mesh filename=/home/mr_robot/test_ws/src/bobo_simulation/simulation_packa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; visual mesh filename=/home/mr_robot/test_ws/src/bobo_simulation/simulation_packa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
- link right_wheel_link: mass 0.01 -> 1.1347; geometry collision mesh filename=/home/mr_robot/test_ws/src/bobo_simulation/simulation_packa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; visual mesh filename=/home/mr_robot/test_ws/src/bobo_simulation/simulation_packa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
Joints:
- joint back_caster_ball_joint: origin xyz=-0.16676 0 0.01 rpy=0 0 0 -> xyz=-0.16676 0 0.025 rpy=0 0 0
- joint front_caster_ball_joint: origin xyz=0.16676 0 0.01 rpy=0 0 0 -> xyz=0.16676 0 0.025 rpy=0 0 0
- joint left_wheel_joint: axis 0 0 1 -> 0 1 0; origin xyz=0.00 0.1665 0.05 rpy=-1.5707963267948966 0 0 -> xyz=-0.000500000000000396 0.179709309933579 0.085 rpy=0 0 0
- joint right_wheel_joint: axis 0 0 1 -> 0 1 0; origin xyz=0.00 -0.1665 0.05 rpy=-1.5707963267948966 0 0 -> xyz=-0.000499999999999182 -0.179709309933579 0.085 rpy=0 0 0

File: simulation_packages/romrobots_description/urdf/yoyo_ros2_control.xacro (robot description, xacro)
@@ -26,5 +26,5 @@
             <robot_param>robot_description</robot_param>
             <robot_param_node>robot_state_publisher</robot_param_node>
-            <parameters>/home/mr_robot/test_ws/src/bobo_simulation/simulation_packages/romrobots_description/config/bobo_controllers.yaml</parameters>
+            <parameters>/home/mr_robot/test_ws/src/bobo_simulation/simulation_packages/romrobots_description/config/yoyo_controllers.yaml</parameters>
             <!-- Output -->
             <odometry_frame>odom</odometry_frame>
@@ -37,5 +37,5 @@
     <gazebo reference="left_wheel_link">
       <material>Gazebo/Black</material>
-      <!-- <kp>1000000.0</kp>
+      <kp>1000000.0</kp>
       <kd>10.0</kd>
       <mu1>1.2</mu1>
@@ -43,7 +43,21 @@
       <fdir1>1 0 0</fdir1>
       <maxVel>0.5</maxVel>
-      <minDepth>0.00</minDepth> -->
+      <minDepth>0.00</minDepth>
+      <!-- <mu1>1.3</mu1>
+      <mu2>1.3</mu2> -->
     </gazebo>
     <gazebo reference="right_wheel_link">
+      <material>Gazebo/Black</material>
+      <kp>1000000.0</kp>
+      <kd>10.0</kd>
+      <mu1>1.2</mu1>
+      <mu2>1.2</mu2>
+      <fdir1>1 0 0</fdir1>
+      <maxVel>0.5</maxVel>
+      <minDepth>0.00</minDepth>
+      <!-- <mu1>1.3</mu1>
+      <mu2>1.3</mu2> -->
+    </gazebo>
+     <gazebo reference="caster_front_link">
       <material>Gazebo/Black</material>
       <!-- <kp>1000000.0</kp>
@@ -54,14 +68,18 @@
       <maxVel>0.5</maxVel>
       <minDepth>0.00</minDepth> -->
-    </gazebo>
-     <gazebo reference="caster_front_link">
-      <material>Gazebo/Black</material>
-      <!-- <mu1>1.0</mu1>
-      <mu2>0.05</mu2> -->
+      <mu1>1.0</mu1>
+      <mu2>0.05</mu2>
     </gazebo>
     <gazebo reference="caster_back_link">
       <material>Gazebo/Black</material>
-      <!-- <mu1>1.0</mu1>
-      <mu2>0.05</mu2> -->
+      <!-- <kp>1000000.0</kp>
+      <kd>10.0</kd>
+      <mu1>1.2</mu1>
+      <mu2>1.2</mu2>
+      <fdir1>1 0 0</fdir1>
+      <maxVel>0.5</maxVel>
+      <minDepth>0.00</minDepth> -->
+      <mu1>1.0</mu1>
+      <mu2>0.05</mu2>
     </gazebo>
     <gazebo reference="imu_link">
