Commit message: sim_pkg OK

File: simulation_packages/romrobots_description/urdf/yoyo.urdf (robot description, URDF)
Before this commit: robot yoyo_standalone, 10 links, 9 joints
Joints:
- joint back_caster_ball_joint: origin xyz=-0.16676 0 0.025 rpy=0 0 0 -> xyz=-0.16676 0 0.0210 rpy=0 0 0
- joint front_caster_ball_joint: origin xyz=0.16676 0 0.025 rpy=0 0 0 -> xyz=0.16676 0 0.0210 rpy=0 0 0

File: simulation_packages/romrobots_description/urdf/yoyo.xacro (robot description, xacro)
@@ -178,5 +178,5 @@
     <parent link="base_link"/>
     <child link="front_caster_ball"/>
-    <origin xyz="0.16676 0 0.025" rpy="0 0 0"/>  <!-- z axis 0.02 နဲ့ 0.03 ကြား -->
+    <origin xyz="0.16676 0 0.0210" rpy="0 0 0"/>  <!-- z axis -->
   </joint>
   <link name="back_caster_ball">
@@ -202,5 +202,5 @@
     <parent link="base_link"/>
     <child link="back_caster_ball"/>
-    <origin xyz="-0.16676 0 0.025" rpy="0 0 0"/>  <!-- z axis 0.02 နဲ့ 0.03 ကြား -->
+    <origin xyz="-0.16676 0 0.0210" rpy="0 0 0"/>  <!-- z axis -->
   </joint>
   <!-- ROM ADD -->
